File: experiments/si4706_radio_eval/radio.kicad_sch (KiCad schematic)
At the start: 35 parts, among them J1 Header, J2 I2C, Q1 BSD840NH6327XTSA1, SW1 Voltage Selector, U1 Si4706-D50-GM, U2 MIC5504-3.3YM5, Y1 32.786kHz

Commit message: radiocore: redesign the Si4706 experiment to a new clock controller with ESP32-C3 and RTC
Other:
- note added: "Instead, GPIO1/2 are strapping pins (see Table 11): for 2-Wire (I2C) pull GPIO1 high and GPIO2 low."
- note added: "Note from the future: always use 3.3V."
- note added: "Note from the future: should provision a three-element Pi matching circuit (two C, one L). Had good results with 20pF, ferrite bead and 220pF net."
- note added: "This part is wrong as shown! pull ~{RST} HIGH to enable chip! ~{SEN} does not enable I2C but selects addr (low: 0x11/17, high: 0x63/99)"
- note removed: "pull ~{RST} low to enable chip and ~{SEN} high to enable I2C"
Changed lines of the file:
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@@
 (kicad_sch
-	(version 20231120)
+	(version 20250114)
 	(generator "eeschema")
-	(generator_version "8.0")
+	(generator_version "9.0")
 	(paper "A4")
+	(text "Note from the future: always use 3.3V."
+		(exclude_from_sim no)
+		(at 247.904 99.06 0)
+		(effects
+			(font
+				(size 1.27 1.27)
+			)
+		)
+	)
+	(text "Simple linear regulator\nfor a safe 3.3V supply."
+		(exclude_from_sim no)
+		(at 244.094 26.162 0)
+		(effects
+			(font
+				(size 1.27 1.27)
+			)
+		)
+	)
+	(text "crystal oscillator"
+		(exclude_from_sim no)
+		(at 59.436 108.966 0)
+		(effects
+			(font
+				(size 1.27 1.27)
+			)
+		)
+	)
+	(text "Qwiic / StemmaQT compat.\nUse regulator with this connector."
+		(exclude_from_sim no)
+		(at 178.562 137.16 90)
+		(effects
+			(font
+				(size 1.27 1.27)
+			)
+		)
+	)
+	(text "compatible with the\nSparkfun Si470x-breakout"
+		(exclude_from_sim no)
+		(at 34.798 158.242 90)
+		(effects
+			(font
+				(size 1.27 1.27)
+			)
+		)
+	)
+	(text "Audio"
+		(exclude_from_sim no)
+		(at 110.998 60.96 0)
+		(effects
+			(font
+				(size 1.27 1.27)
+			)
+			(justify left)
+		)
+	)
+	(text "You're not supposed to populate / use all of\nthese antennas. It is a development board to\nsee which / if one works well."
+		(exclude_from_sim no)
+		(at 148.336 37.338 0)
+		(effects
+			(font
+				(size 1.27 1.27)
+			)
+		)
+	)
+	(text "I2C"
+		(exclude_from_sim no)
+		(at 56.642 63.754 0)
+		(effects
+			(font
+				(size 1.27 1.27)
+			)
+			(justify right)
+		)
+	)
+	(text "Select which voltage to supply\nto the chip. See notes on J1 and J2."
+		(exclude_from_sim no)
+		(at 247.65 68.834 0)
+		(effects
+			(font
+				(size 1.27 1.27)
+			)
+		)
+	)
+	(text "Check AN383 for Antenna Design\n- §5.2 has information on selecting proper L\n  and monitoring internal varactor with READANTCAP\n- Appendix B has information on calculation; value\n  of 120nH is recommended in general though"
+		(exclude_from_sim no)
+		(at 142.494 76.2 0)
+		(effects
+			(font
+				(size 1.27 1.27)
+			)
+			(justify left)
+		)
+	)
+	(text "Note from the future: should provision a\nthree-element Pi matching circuit (two C, one L).\nHad good results with 20pF, ferrite bead and 220pF net."
+		(exclude_from_sim no)
+		(at 189.738 56.388 0)
+		(effects
+			(font
+				(size 1.27 1.27)
+			)
+		)
+	)
+	(text "device"
+		(exclude_from_sim no)
+		(at 225.044 146.05 0)
+		(effects
+			(font
+				(size 1.27 1.27)
+			)
+		)
+	)
+	(text "When using this header, use 3.3V ONLY\nand switch the voltage selector to VBUS\n(bypassing the regulator). Otherwise you\nmight damage the IO pins with overvoltage."
+		(exclude_from_sim no)
+		(at 88.9 158.496 90)
+		(effects
+			(font
+				(size 1.27 1.27)
+			)
+		)
+	)
+	(text "This part is wrong as shown!\n\npull ~{RST} HIGH to enable chip!\n\n~{SEN} does not enable I2C but selects addr\n(low: 0x11/17, high: 0x63/99)"
+		(exclude_from_sim no)
+		(at 40.64 26.162 0)
+		(effects
+			(font
+				(size 1.27 1.27)
+			)
+		)
+	)
+	(text "connector"
+		(exclude_from_sim no)
+		(at 241.3 146.05 0)
+		(effects
+			(font
+				(size 1.27 1.27)
+			)
+		)
+	)
+	(text "VA: 2.7–5.5V\nVD: 1.6–3.6V\nsafe: 3.3V"
+		(exclude_from_sim no)
+		(at 82.55 24.384 0)
+		(effects
+			(font
+				(size 1.27 1.27)
+			)
+		)
+	)
+	(text "optional"
+		(exclude_from_sim no)
+		(at 264.922 87.884 0)
+		(effects
+			(font
+				(size 1.27 1.27)
+			)
+		)
+	)
+	(text "GPIO"
+		(exclude_from_sim no)
+		(at 56.134 72.644 0)
+		(effects
+			(font
+				(size 1.27 1.27)
+			)
+			(justify right)
+		)
+	)
+	(text "MOSFET Level Shifting for I2C\n* NXP AppNote AN10441\n* https://electronics.stackexchange.com/a/367055"
+		(exclude_from_sim no)
+		(at 221.742 120.142 0)
+		(effects
+			(font
+				(size 1.27 1.27)
+			)
+			(justify left bottom)
+		)
+	)
+	(text "VCC ≤ VBUS !"
+		(exclude_from_sim no)
+		(at 254.508 116.84 0)
+		(effects
+			(font
+				(size 1.27 1.27)
+				(thickness 0.254)
+				(bold yes)
+			)
+			(justify left bottom)
+		)
+	)
+	(text "Instead, GPIO1/2 are strapping pins\n(see Table 11): for 2-Wire (I2C)\npull GPIO1 high and GPIO2 low."
+		(exclude_from_sim no)
+		(at 33.274 71.882 0)
+		(effects
+			(font
+				(size 1.27 1.27)
+			)
+		)
+	)
 	(junction
 		(at 90.17 35.56)
@@
 		)
 	)
-	(text "Simple linear regulator\nfor a safe 3.3V supply."
-		(exclude_from_sim no)
-		(at 244.094 26.162 0)
-		(effects
-			(font
-				(size 1.27 1.27)
-			)
-		)
-	)
-	(text "crystal oscillator"
-		(exclude_from_sim no)
-		(at 59.436 108.966 0)
-		(effects
-			(font
-				(size 1.27 1.27)
-			)
-		)
-	)
-	(text "Qwiic / StemmaQT compat.\nUse regulator with this connector."
-		(exclude_from_sim no)
-		(at 178.562 137.16 90)
-		(effects
-			(font
-				(size 1.27 1.27)
-			)
-		)
-	)
-	(text "compatible with the\nSparkfun Si470x-breakout"
-		(exclude_from_sim no)
-		(at 34.798 158.242 90)
-		(effects
-			(font
-				(size 1.27 1.27)
-			)
-		)
-	)
-	(text "Audio"
-		(exclude_from_sim no)
-		(at 110.998 60.96 0)
-		(effects
-			(font
-				(size 1.27 1.27)
-			)
-			(justify left)
-		)
-	)
-	(text "You're not supposed to populate / use all of\nthese antennas. It is a development board to\nsee which / if one works well."
-		(exclude_from_sim no)
-		(at 148.336 37.338 0)
-		(effects
-			(font
-				(size 1.27 1.27)
-			)
-		)
-	)
-	(text "I2C"
-		(exclude_from_sim no)
-		(at 56.642 63.754 0)
-		(effects
-			(font
-				(size 1.27 1.27)
-			)
-			(justify right)
-		)
-	)
-	(text "Select which voltage to supply\nto the chip. See notes on J1 and J2."
-		(exclude_from_sim no)
-		(at 247.65 68.834 0)
-		(effects
-			(font
-				(size 1.27 1.27)
-			)
-		)
-	)
-	(text "Check AN383 for Antenna Design\n- §5.2 has information on selecting proper L\n  and monitoring internal varactor with READANTCAP\n- Appendix B has information on calculation; value\n  of 120nH is recommended in general though"
-		(exclude_from_sim no)
-		(at 142.494 76.2 0)
-		(effects
-			(font
-				(size 1.27 1.27)
-			)
-			(justify left)
-		)
-	)
-	(text "device"
-		(exclude_from_sim no)
-		(at 225.044 146.05 0)
-		(effects
-			(font
-				(size 1.27 1.27)
-			)
-		)
-	)
-	(text "When using this header, use 3.3V ONLY\nand switch the voltage selector to VBUS\n(bypassing the regulator). Otherwise you\nmight damage the IO pins with overvoltage."
-		(exclude_from_sim no)
-		(at 88.9 158.496 90)
-		(effects
-			(font
-				(size 1.27 1.27)
-			)
-		)
-	)
-	(text "pull ~{RST} low to enable chip\nand ~{SEN} high to enable I2C"
-		(exclude_from_sim no)
-		(at 30.988 46.736 90)
-		(effects
-			(font
-				(size 1.27 1.27)
-			)
-		)
-	)
-	(text "connector"
-		(exclude_from_sim no)
-		(at 241.3 146.05 0)
-		(effects
-			(font
-				(size 1.27 1.27)
-			)
-		)
-	)
-	(text "VA: 2.7–5.5V\nVD: 1.6–3.6V\nsafe: 3.3V"
-		(exclude_from_sim no)
-		(at 82.55 24.384 0)
-		(effects
-			(font
-				(size 1.27 1.27)
-			)
-		)
-	)
-	(text "optional"
-		(exclude_from_sim no)
-		(at 264.922 87.884 0)
-		(effects
-			(font
-				(size 1.27 1.27)
-			)
-		)
-	)
-	(text "GPIO"
-		(exclude_from_sim no)
-		(at 56.134 72.644 0)
-		(effects
-			(font
-				(size 1.27 1.27)
-			)
-			(justify right)
-		)
-	)
-	(text "MOSFET Level Shifting for I2C\n* NXP AppNote AN10441\n* https://electronics.stackexchange.com/a/367055"
-		(exclude_from_sim no)
-		(at 221.742 120.142 0)
-		(effects
-			(font
-				(size 1.27 1.27)
-			)
-			(justify left bottom)
-		)
-	)
-	(text "VCC ≤ VBUS !"
-		(exclude_from_sim no)
-		(at 254.508 116.84 0)
-		(effects
-			(font
-				(size 1.27 1.27)
-				(thickness 0.254)
-				(bold yes)
-			)
-			(justify left bottom)
-		)
-	)
 	(global_label "~{RST}"
 		(shape input)
@@
 		)
 	)
+	(embedded_fonts no)
 )
